File: PCB/Cabinas/Cabinas.kicad_pcb (KiCad board)
At the start: 2 copper layers, 196.7 x 93.5 mm, 113 parts, among them J1 JACK_ST_3SW, K1 CONN_3, M1 WTV020-SD, P1 CONN_2, P10 CONN_2, P11 CONN_2, P12 CONN_2, P13 DIN_5, P2 CONN_2, P3 CONN_2, P4 CONN_2, P5 CONN_2, P6 CONN_2, P7 CONN_2, P8 CONN_2, P9 CONN_2, Q1 MOSFET_N, Q10 MOSFET_N, Q11 MOSFET_N, Q12 MOSFET_N, Q2 MOSFET_N, Q3 MOSFET_N, Q4 MOSFET_N, Q5 MOSFET_N, Q6 MOSFET_N, Q7 MOSFET_N, Q8 MOSFET_N, Q9 MOSFET_N, SW1 PUSHBUTTON, SW10 PUSHBUTTON, SW11 PUSHBUTTON, SW12 PUSHBUTTON, SW2 PUSHBUTTON, SW3 PUSHBUTTON, SW4 PUSHBUTTON, SW5 PUSHBUTTON, SW6 PUSHBUTTON, SW7 PUSHBUTTON, SW8 PUSHBUTTON, SW9 PUSHBUTTON, U1 BTM, U2 7805, U3 TL072

Commit message: Rev 1.2
Rev 1.2
Parts:
- removed P10, P11, P12, P9: CONN_2, PIN_ARRAY_2X1
- added C13: 470uF, CAP_8_3.5, F.Cu at (222.5, 130.3)
- added GS1: GS3, GS3, F.Cu at (207.8, 141.0)
- added GS2: GS3, GS3, F.Cu at (188.5, 121.9)
- added U4: 74HC595, DIP-16__300, F.Cu at (139.2, 109.7)
- added U5: 74HC595, DIP-16__300, F.Cu at (109.7, 117.9)
- C7: footprint C1V5 -> CAP_8_3.5
- P1, P2, P3, P4, P5, P6, P7, P8: value CONN_2 -> CONN_4; footprint PIN_ARRAY_2X1 -> PIN_ARRAY_CAB
- moved P7 59.6 mm to (70.6, 63.0)
- moved P8 57.4 mm to (55.6, 63.0)
- moved P5 39.8 mm to (120.9, 62.5)
- moved P6 39.0 mm to (106.4, 62.5)
- moved P3 25.8 mm to (170.2, 62.5)
- moved P4 25.0 mm to (153.4, 62.5)
- moved P1 11.8 mm to (217.4, 63.0)
- moved P2 11.0 mm to (201.7, 63.0)
- moved C6 2.67 mm to (197.4, 135.4)
- moved R3 0.28 mm to (191.5, 84.8)
Connections:
- A1 pad 10: D7 -> SR_OE
- A1 pad 11: D8 -> SR_LCLK
- A1 pad 12: D9 -> SR_CLK
- A1 pad 15: MP3_CK -> (no net)
- A1 pad 16: MP3_RESET -> (no net)
- A1 pad 17: D10 -> (no net)
- A1 pad 18: D11 -> (no net)
- A1 pad 19: D12 -> (no net)
- A1 pad 20: D13 -> (no net)
- A1 pad 23: MP3_BUSY -> (no net)
- A1 pad 24: MP3_DATA -> (no net)
- A1 pad 5: D2 -> MP3_RESET
- A1 pad 6: D3 -> MP3_CK
- A1 pad 7: D4 -> MP3_DATA
- A1 pad 8: D5 -> MP3_BUSY
- A1 pad 9: D6 -> SR_Input
- C3 pad 2: N-0000046 -> GND
- C4 pad 2: N-0000046 -> GND
- C5 pad 2: N-0000046 -> GND
- C6 pad 2: N-0000046 -> GND
- C7 pad 2: N-0000046 -> GND
- D1 pad 1: N-0000024 -> N-0000047
- D13 pad 1: N-0000016 (its old number) -> N-0000012
- D14 pad 1: N-0000012 -> N-0000015
- D15 pad 1: N-0000013 (its old number) -> N-000004
- D16 pad 1: N-0000054 (its old number) -> N-000008
- D17 pad 1: N-0000057 (its old number) -> N-0000022
- D18 pad 1: N-0000052 (its old number) -> N-0000023
- D2 pad 1: N-0000035 -> N-0000024
- D3 pad 1: N-0000031 -> N-0000028
- D4 pad 1: N-000006 (its old number) -> N-0000056
- D5 pad 1: N-000009 -> N-0000050
- D6 pad 1: N-000001 (its old number) -> N-0000053
- ELEC1 pad 2: Vbias -> N-0000077
- M1 pad 5: Vbias -> N-0000068
- P1 pad 1: +12V -> N-0000047
- P2 pad 1: +12V -> N-0000047
- P2 pad 2: N-0000035 -> N-0000024
- P3 pad 1: +12V -> N-0000056
- P3 pad 2: N-0000031 -> N-0000050
- P4 pad 1: +12V -> N-0000056
- P4 pad 2: N-000006 (its old number) -> N-0000050
- P5 pad 1: +12V -> N-0000012
- P5 pad 2: N-000009 -> N-0000015
- P6 pad 1: +12V -> N-0000012
- P6 pad 2: N-000001 (its old number) -> N-0000015
- P7 pad 1: +12V -> N-000008
- P7 pad 2: N-0000016 (its old number) -> N-0000022
- P8 pad 1: +12V -> N-000008
- P8 pad 2: N-0000012 -> N-0000022
- Q1 pad D: N-0000024 -> N-0000047
- Q10 pad D: N-0000054 (its old number) -> N-000008
- Q11 pad D: N-0000057 (its old number) -> N-0000022
- Q12 pad D: N-0000052 (its old number) -> N-0000023
- Q2 pad D: N-0000035 -> N-0000024
- Q3 pad D: N-0000031 -> N-0000028
- Q4 pad D: N-000006 (its old number) -> N-0000056
- Q5 pad D: N-000009 -> N-0000050
- Q6 pad D: N-000001 (its old number) -> N-0000053
- Q7 pad D: N-0000016 (its old number) -> N-0000012
- Q8 pad D: N-0000012 -> N-0000015
- Q9 pad D: N-0000013 (its old number) -> N-000004
- SW1 pad 2: D2 -> 1
- SW10 pad 2: D11 -> 10
- SW11 pad 2: D12 -> 11
- SW12 pad 2: D13 -> 12
- SW2 pad 2: D3 -> 2
- SW3 pad 2: D4 -> 3
- SW4 pad 2: D5 -> 4
- SW5 pad 2: D6 -> 5
- SW6 pad 2: D7 -> 6
- SW7 pad 2: D8 -> 7
- SW8 pad 2: D9 -> 8
- SW9 pad 2: D10 -> 9
Routing:
- net D13: track 109.0 -> 0.00 mm
- net D2: track 105.2 -> 0.00 mm
- net 1: track 0.00 -> 92.7 mm
- net D12: track 91.9 -> 0.00 mm
- net D3: track 91.5 -> 0.00 mm
- net D4: track 77.7 -> 0.00 mm
- net D11: track 73.1 -> 0.00 mm
- net +5V: track 460.2 -> 531.5 mm, vias 5 -> 7
- net 2: track 0.00 -> 70.7 mm
- net N-0000046: track 69.9 -> 0.00 mm
- net D5: track 63.4 -> 0.00 mm
- net 12: track 0.00 -> 62.9 mm
- net 3: track 0.00 -> 57.1 mm
- net D10: track 50.9 -> 0.00 mm
- net D6: track 47.8 -> 0.00 mm
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Other:
- board text added: "+5v"
- board text added: "22"
- board text added: "23"
- board text added: "24"
- board text added: "25"
- board text added: "Grupo A DB-2"
- board text added: "Grupo B DB-1"
- board text added: "Grupo C DB-1"
- board text added: "Grupo D DB-1"
- board text added: "Grupo F DB-2"
- board text added: "Grupo G DB-2"
- board text added: "Grupo H DB-1"
- board text added: "Grupo I DB-2"
- board text added: "Rx"
- board text added: "Signal"
- board text added: "Tx"

Commit message: BOM
BOM
Parts:
- U1: value BTM -> BTM_2; footprint btm -> btm_2
- U4, U5: footprint DIP-16__300 -> ShiftReg
- moved C1 7.04 mm to (56.1, 127.3)
- moved C12 5.17 mm to (190.2, 109.5)
Connections:
- R15 pad 2: GND -> A1 (TX)
- R16 pad 1: A1 (TX) -> GND
- R17 pad 2: GND -> A1 (TX)
- U1 pad 4: +5V -> GND
- U1 pad 5: (no net) -> +5V
- U1 pad 6: GND -> (no net)
Routing:
- net A1 (TX): track 25.7 -> 31.8 mm
- net GND: track 4.08 -> 9.90 mm
- net MP3_OUTPUT: track 14.7 -> 20.3 mm
- net +12V: track 277.3 -> 279.5 mm
- net N-0000067: track 2.59 -> 4.50 mm
- net +5V: track 531.5 -> 530.6 mm
Other:
- board text added: "Busy"
- board text added: "CLK"
- board text added: "Data"
- board text added: "Reset"
- board text added: "Rev 1.2"
- board text removed: "+5v"
- board text removed: "Rev 1.0"
- board text removed: "Rx"
- board text removed: "Tx"

Commit message: PCB Rev 1.3
Parts:
- removed the 3.5mm_Screw at (136.0, 83.2)
- removed the 3.5mm_Screw at (45.6, 144.7)
- removed the 3.5mm_Screw at (231.1, 144.7)
- removed C11, C12: 1uF, C1V5
- removed C8: 47uF, C1V5
- removed ELEC1: ELECTRET_MIC_SUP, pin_array_3x2
- removed GS1, GS2: GS3, GS3
- removed J1: JACK_ST_3SW, pin_array_3x2
- removed JP1: JUMPER, PIN_ARRAY_2X1
- removed R18, R19, R21, R22, R23, R24, R26: 10k, R3
- removed R20: 270k, R3
- removed R25: 2.2k, R3
- removed U3: TL072, DIP-8__300_ELL
- added 3.5mm_Screw: VAL**, 3.5mm_Screw, F.Cu at (233.0, 144.8)
- added 3.5mm_Screw: VAL**, 3.5mm_Screw, F.Cu at (45.7, 144.8)
- added 3.5mm_Screw: VAL**, 3.5mm_Screw, F.Cu at (233.0, 65.4)
- added 3.5mm_Screw: VAL**, 3.5mm_Screw, F.Cu at (45.7, 65.4)
- added D25: DIODE, D3, F.Cu at (56.1, 134.9)
- added FB1: FILTER, PIN_ARRAY_2X1, F.Cu at (133.3, 138.4)
- added K2: CONN_3, PIN_ARRAY_3X1, F.Cu at (204.5, 107.3)
- added SW13: PUSHBUTTON, TactileSW_2, F.Cu at (196.8, 113.7)
- added SW14: PUSHBUTTON, TactileSW_2, F.Cu at (196.8, 121.9)
- added SW15: PUSHBUTTON, TactileSW_2, F.Cu at (196.8, 130.2)
- added TP1: CONN_3, PIN_ARRAY_3X1, F.Cu at (190.1, 109.3)
- added TP2: CONN_2, PIN_ARRAY_2X1, F.Cu at (68.6, 110.2)
- added TP3: CONN_2, PIN_ARRAY_2X1, F.Cu at (170.2, 108.1)
- C4, C5: footprint C1 -> C1V5
- moved C6 37.9 mm to (223.2, 107.7), turned to 0 degrees
- moved C7 37.7 mm to (223.2, 117.0), turned to 0 degrees
- moved U4 6.87 mm to (132.4, 108.7)
- moved U1 5.08 mm to (128.9, 142.2)
- moved C4 3.78 mm to (146.4, 139.9)
Connections:
- M1 pad 12: (no net) -> Next
- M1 pad 2: (no net) -> MP3_OUTPUT
- M1 pad 4: MP3_OUTPUT -> N-0000043
- M1 pad 5: N-0000063 -> (no net)
- M1 pad 9: (no net) -> Play
- P13 pad 4: N-0000017 (its old number) -> +5V
- P13 pad 5: +12V -> (no net)
- U1 pad 5: +5V -> N-0000046
Routing:
- net Vbias: track 60.7 -> 0.00 mm, vias 1 -> 0
- net GND: track 9.90 -> 56.1 mm, vias 2 -> 0
- net +3.3V: track 17.8 -> 62.0 mm, vias 0 -> 2
- net +12V: track 279.5 -> 235.9 mm, vias 9 -> 4
- net Play: track 0.00 -> 36.9 mm
- net Next: track 0.00 -> 35.3 mm
- net N-0000076: track 30.7 -> 0.00 mm
- net N-0000048: track 12.2 -> 42.1 mm, vias 0 -> 1
- net N-0000017 (its old number): track 29.1 -> 0.00 mm
- net N-0000065: track 26.0 -> 0.00 mm, vias 2 -> 0
- net MP3_OUTPUT: track 20.3 -> 43.0 mm, vias 0 -> 3
- net N-0000043: track 0.00 -> 19.4 mm, vias 0 -> 2
- net MP3_RESET: track 56.2 -> 74.8 mm
- net N-0000064: track 18.4 -> 0.00 mm
- net N-0000074: track 18.1 -> 0.00 mm
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Other:
- board text added: "+3.3V"
- board text added: "+5V"
- board text added: "Audio"
- board text added: "B"
- board text added: "G"
- board text added: "MP3 Output"
- board text added: "MP3 Speaker"
- board text added: "Next"
- board text added: "Play/Stop"
- board text added: "R"
- board text added: "Rev 1.3"
- board text added: "SCL A4"
- board text added: "SDA A5"
- board text removed: "Rev 1.2"
- board text removed: "Signal"

Commit message: Rev 1.4
Parts:
- removed K1: CONN_3, bornier3
- removed K2: CONN_3, PIN_ARRAY_3X1
- added C11: 0.022uF, C1, F.Cu at (214.0, 117.2)
- added C12: 0.1uF, C1, F.Cu at (214.0, 121.5)
- added C14: 10uF, CAP_8_3.5, F.Cu at (204.8, 132.0)
- added C15: 270uF, CAP_8_3.5, F.Cu at (195.0, 132.0)
- added C16: 0.1uF, C1, F.Cu at (196.8, 120.0)
- added C17: 270uF, CAP_8_3.5, F.Cu at (186.5, 120.5)
- added C8: 0.22uF, C1, F.Cu at (212.0, 111.5)
- added J1: JACK_ST, PIN_ARRAY_3X1, F.Cu at (204.5, 108.5)
- added J2: JACK_ST, Jack_Pin_3, F.Cu at (182.2, 108.5)
- added P10: CONN_2, PINHEAD1-2, F.Cu at (234.0, 132.8)
- added P11: CONN_6, PINHEAD1-6, F.Cu at (204.0, 140.0)
- added P9: CONN_2, PINHEAD1-2, F.Cu at (234.0, 109.8)
- added R18: 220, R1, F.Cu at (216.8, 110.0)
- added R19: 2.2k, R1, F.Cu at (216.8, 113.0)
- added R20: 10R, R1, F.Cu at (193.2, 123.0)
- added R21: R, R1, F.Cu at (175.2, 132.2)
- added R22: R, R1, F.Cu at (175.2, 127.5)
- added R23: R, R1, F.Cu at (179.8, 124.0)
- added R24: 10k, R1, F.Cu at (186.5, 142.0)
- added R25: 10k, R1, F.Cu at (181.0, 142.0)
- added RV1: 10k, PIN_ARRAY_3X1, F.Cu at (219.5, 119.0)
- added U3: LM386, DIP-8__300_ELL, F.Cu at (204.5, 122.2)
- added U6: TL082, DIP-8__300_ELL, F.Cu at (183.5, 131.5)
- FB1: footprint PIN_ARRAY_2X1 -> R3
- P13: footprint MIDI -> PIN_ARRAY_4x1
- R13, R14, R15, R16, R17: footprint R3 -> R1
- U1: footprint btm_2 -> btm_3
- moved R17 40.8 mm to (110.0, 144.0), turned to 270 degrees
- moved R15 38.0 mm to (112.5, 144.2), turned to 90 degrees
- moved C3 37.3 mm to (133.0, 133.0), turned to 180 degrees
- moved A1 35.2 mm to (98.5, 127.8)
- moved R16 35.0 mm to (115.5, 144.0), turned to 270 degrees
- moved FB1 34.6 mm to (98.8, 140.2)
- moved U1 30.2 mm to (98.8, 144.0), turned to 0 degrees
- moved SW15 29.8 mm to (167.5, 135.2)
- moved SW13 29.6 mm to (167.2, 113.8)
- moved M1 29.5 mm to (143.2, 123.8)
- moved REG1 29.5 mm to (131.0, 139.3)
- moved TP1 29.5 mm to (160.6, 109.3)
- moved TP3 29.5 mm to (140.7, 108.1)
- moved SW14 29.4 mm to (167.5, 124.2)
- moved C9 28.2 mm to (132.5, 146.0), turned to 0 degrees
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Connections:
- C1 pad 1: +12V -> +12P
- D25 pad 2: +12V -> +12P
- P13 pad 1: I2CSCL -> I2CSDA
- P13 pad 2: I2CSDA -> I2CSCL
- P13 pad 5: (no net) -> GND
- R15 pad 1: N-0000040 (its old number) -> N-0000014
- R16 pad 2: N-0000040 (its old number) -> N-0000014
- R17 pad 1: N-0000040 (its old number) -> A1 (TX)
- R17 pad 2: A1 (TX) -> N-0000014
- U1 pad 2: N-0000040 (its old number) -> N-0000014
- U2 pad Vi: +12V -> +12P
Routing:
- net +12P: track 0.00 -> 293.3 mm
- net +12V: track 235.9 -> 30.0 mm, vias 4 -> 0
- net MIC_PREAMP: track 0.00 -> 64.3 mm, vias 0 -> 2
- net +5V: track 513.6 -> 462.5 mm, vias 8 -> 3
- net I2CSCL: track 99.1 -> 56.4 mm, vias 0 -> 1
- net Vbias: track 0.00 -> 38.5 mm
- net GND: track 56.1 -> 17.7 mm
- net I2CSDA: track 83.9 -> 59.2 mm, vias 3 -> 0
- net 1: track 98.8 -> 123.1 mm
- net N-0000053: track 0.00 -> 23.8 mm, vias 0 -> 1
- net 6: track 20.5 -> 44.2 mm
- net 4: track 48.3 -> 71.7 mm
- net 5: track 33.6 -> 57.0 mm
- net 2: track 76.7 -> 99.9 mm, vias 1 -> 0
- net N-0000040 (its old number): track 22.9 -> 0.00 mm
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- added copper zone on F.Cu, net +12V
Other:
- rule trace_min: 0.254 -> 0.01
- rule via_min_size: 0.889 -> 0.035
- board text added: "+"
- board text added: "-"
- board text added: "Hackerspace Cholula"
- board text added: "LM386"
- board text added: "Mic"
- board text added: "Out"
- board text added: "Pre"
- board text added: "Rev 1.4"
- board text added: "SCL A5"
- board text added: "SDA A4"
- board text added: "TL072"
- board text added: "Vb"
- board text added: "Vbias"
- board text removed: "Bluetooth Module"
- board text removed: "Bottom"
- board text removed: "Rev 1.3"
- board text removed: "SCL A4"
- board text removed: "SDA A5"
- board text removed: "Top"

Commit message: Rev 1.4
Changed lines of the file:
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@@
   )
   (setup
-    (last_trace_width 0.381)
+    (last_trace_width 0.254)
     (user_trace_width 0.3048)
     (user_trace_width 0.381)
@@
     )
   )
+  (gr_line (start 72.75 132) (end 75 132) (angle 90) (layer F.SilkS) (width 0.2))
   (gr_text Pre (at 213.8 140) (layer F.SilkS)
     (effects (font (size 1.5 1.5) (thickness 0.3)))
@@
   (gr_line (start 65 125) (end 67 125) (angle 90) (layer F.SilkS) (width 0.2))
   (gr_line (start 75 132) (end 76 131) (angle 90) (layer F.SilkS) (width 0.2))
-  (gr_line (start 73 132) (end 75 132) (angle 90) (layer F.SilkS) (width 0.2))
-  (gr_line (start 72 131) (end 73 132) (angle 90) (layer F.SilkS) (width 0.2))
+  (gr_line (start 71.75 131) (end 72.75 132) (angle 90) (layer F.SilkS) (width 0.2))
   (gr_line (start 71 129.5) (end 72 128.5) (angle 90) (layer F.SilkS) (width 0.2))
   (gr_line (start 69 129.5) (end 71 129.5) (angle 90) (layer F.SilkS) (width 0.2))
@@
     (effects (font (size 2 2) (thickness 0.3) italic))
   )
-  (gr_text 1 (at 229.87 104.013) (layer F.SilkS)
+  (gr_text 1 (at 222 98.5) (layer F.SilkS)
     (effects (font (size 1.5 1.5) (thickness 0.3)))
   )
-  (gr_text 2 (at 213.36 104.013) (layer F.SilkS)
+  (gr_text 2 (at 205 98.5) (layer F.SilkS)
     (effects (font (size 1.5 1.5) (thickness 0.3)))
   )
-  (gr_text 3 (at 196.85 104.013) (layer F.SilkS)
+  (gr_text 3 (at 188.75 98.5) (layer F.SilkS)
     (effects (font (size 1.5 1.5) (thickness 0.3)))
   )
-  (gr_text 4 (at 171.75 100.25) (layer F.SilkS)
+  (gr_text 4 (at 172 98.5) (layer F.SilkS)
     (effects (font (size 1.5 1.5) (thickness 0.3)))
   )
-  (gr_text 5 (at 154.925 104.263) (layer F.SilkS)
+  (gr_text 5 (at 154.75 98.5) (layer F.SilkS)
     (effects (font (size 1.5 1.5) (thickness 0.3)))
   )

Commit message: Rev 1.5
Audio estereo
Parts:
- removed C10: 1uF, C1V5
- removed C3: 0.1uF, C1
- removed M1: WTV020-SD, MP3
- removed P11: CONN_6, PINHEAD1-6
- removed R23: R, R1
- removed REG1: NPC1700, TO92
- removed TP1: CONN_3, PIN_ARRAY_3X1
- removed TP3: CONN_2, PIN_ARRAY_2X1
- added A2: PROMINI, ProMini, F.Cu at (148.6, 116.6)
- added K1: CONN_3, PIN_ARRAY_3X1, F.Cu at (156.0, 145.5)
- added K2: CONN_3, PIN_ARRAY_3X1, F.Cu at (123.4, 117.6)
- added MP31: VS1053_ADAFRUIT, VS1030_Adafruit, F.Cu at (189.5, 146.8)
- added R26: 10k, R1, F.Cu at (156.7, 140.0)
- added R27: 10k, R1, F.Cu at (148.3, 140.0)
- added R28: 10k, R1, F.Cu at (140.0, 140.0)
- added R29: R, R1, F.Cu at (212.3, 140.7)
- added R30: R, R1, F.Cu at (212.9, 137.7)
- added RV2: 10k, Trimpot, F.Cu at (196.8, 134.4)
- added RV3: 10k, Trimpot, F.Cu at (206.0, 134.4)
- RV1: footprint PIN_ARRAY_3X1 -> Trimpot
- moved SW15 36.0 mm to (131.6, 133.1), turned to 90 degrees
- moved R25 35.2 mm to (216.2, 144.3), turned to 180 degrees
- moved R24 30.1 mm to (216.2, 147.1), turned to 0 degrees
- moved SW14 28.7 mm to (140.2, 133.1), turned to 90 degrees
- moved C15 27.6 mm to (222.2, 127.5), turned to 180 degrees
- moved SW13 27.1 mm to (148.3, 133.1), turned to 90 degrees
- moved R22 23.3 mm to (195.1, 139.7), turned to 180 degrees
- moved R21 22.7 mm to (195.3, 142.7), turned to 0 degrees
- moved U6 22.7 mm to (204.0, 141.2)
- moved J2 13.8 mm to (196.1, 108.2), turned to 180 degrees
- moved C14 10.3 mm to (214.1, 127.8), turned to 270 degrees
- moved C17 9.63 mm to (195.6, 123.7), turned to 270 degrees
- moved R20 6.93 mm to (193.5, 116.1)
- moved SW3 4.71 mm to (194.1, 87.9)
- moved SW4 4.70 mm to (177.0, 87.9)
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Connections:
- A1 pad 5: MP3_RESET -> (no net)
- A1 pad 6: MP3_CK -> (no net)
- A1 pad 7: MP3_DATA -> (no net)
- A1 pad 8: MP3_BUSY -> (no net)
- J2 pad 2: N-0000053 (its old number) -> N-0000070
- J2 pad 3: N-0000053 (its old number) -> N-0000069
- R21 pad 1: MP3_OUTPUT -> ROUT
- R24 pad 1: +12P -> Vbias
- R24 pad 2: Vbias -> +12P
- U6 pad 1: N-0000053 (its old number) -> N-0000069
- U6 pad 5: N-0000029 -> Vbias
- U6 pad 7: N-0000027 (its old number) -> N-0000070
Routing:
- net I2CSCL: track 56.4 -> 135.5 mm, vias 1 -> 2
- net LOUT: track 0.00 -> 67.2 mm, vias 0 -> 3
- net +5V: track 462.5 -> 525.0 mm, vias 3 -> 5
- net +3.3V: track 61.9 -> 0.00 mm, vias 4 -> 0
- net MP3_CK: track 56.7 -> 0.00 mm
- net I2CSDA: track 59.2 -> 114.3 mm, vias 0 -> 1
- net MP3_RESET: track 76.4 -> 21.8 mm, vias 2 -> 0
- net MP3_BUSY: track 46.7 -> 0.00 mm
- net ROUT: track 0.00 -> 45.2 mm
- net N-0000070: track 0.00 -> 44.8 mm, vias 0 -> 2
- net MP3_OUTPUT: track 44.8 -> 0.00 mm, vias 3 -> 0
- net N-0000058: track 0.00 -> 44.3 mm
- net MP3_DATA: track 44.1 -> 0.00 mm
- net N-0000057: track 0.00 -> 40.1 mm
- net N-0000069: track 0.00 -> 39.8 mm
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Other:
- board text added: "L"
- board text added: "NEXT"
- board text added: "PLAY"
- board text added: "RESET"
- board text added: "Rev 1.5"
- board text removed: "+"
- board text removed: "+3.3V"
- board text removed: "-"
- board text removed: "Audio"
- board text removed: "Busy"
- board text removed: "CLK"
- board text removed: "Data"
- board text removed: "MP3 Module"
- board text removed: "MP3 Output"
- board text removed: "MP3 Speaker"
- board text removed: "Next"
- board text removed: "Out"
- board text removed: "Play/Stop"
- board text removed: "Pre"
- board text removed: "Reset"
- board text removed: "Rev 1.4"
- board text removed: "TL072"
- board text removed: "Vb"
- board text removed: "Vbias"

Commit message: Firmware V3.0
Parts:
- removed C11: 0.022uF, C1
- removed C16: 0.1uF, C1
- removed C17: 270uF, CAP_8_3.5
- removed R20: 10R, R1
- added C3: 10uF, C1V5, F.Cu at (214.4, 119.6)
- added P11: CONN_2, PIN_ARRAY_2X1, F.Cu at (197.1, 124.0)
- C12: value 0.1uF -> 10pF
- C8: value 0.22uF -> 10uF; footprint C1 -> C1V5
- R18: value 220 -> 0R
- R19: value 2.2k -> 100
- moved C14 22.2 mm to (195.6, 115.6), turned to 0 degrees
- moved R19 20.2 mm to (218.7, 133.1), turned to 135 degrees
- moved C8 15.5 mm to (213.1, 127.0), turned to 0 degrees
- moved RV1 12.6 mm to (214.1, 106.9), turned to 0 degrees
- moved C12 10.1 mm to (214.1, 131.6)
- moved R18 7.44 mm to (211.1, 114.8), turned to 0 degrees
- moved U3 0.80 mm to (205.0, 121.4), turned to 270 degrees
Connections:
- C12 pad 1: N-0000066 -> N-0000064
- C12 pad 2: N-0000065 -> N-0000063
- C14 pad 2: N-0000063 -> N-0000062
- C8 pad 1: N-0000060 (its old number) -> N-0000063
- C8 pad 2: GND -> MIC_PREAMP
- J1 pad 3: N-0000054 (its old number) -> N-0000069
- MP31 pad 26: (no net) -> +5V
- R18 pad 1: N-0000054 (its old number) -> N-0000062
- R18 pad 2: N-0000060 (its old number) -> N-0000061
- R19 pad 1: N-0000060 (its old number) -> GND
- R19 pad 2: N-0000067 (its old number) -> N-0000064
- RV1 pad 1: N-0000067 (its old number) -> N-0000069
- RV1 pad 2: N-0000066 -> N-0000068
- U3 pad 3: N-0000065 -> N-0000068
- U3 pad 5: N-0000062 -> N-0000063
- U3 pad 6: +12P -> +12V
- U3 pad 7: (no net) -> N-0000065
- U3 pad 8: N-0000063 -> N-0000061
Routing:
- net +5V: track 525.0 -> 571.8 mm, vias 5 -> 8
- net +12P: track 290.5 -> 256.3 mm, vias 5 -> 1
- net MIC_PREAMP: track 35.7 -> 58.9 mm, vias 3 -> 4
- net N-0000068: track 0.00 -> 19.0 mm
- net +12V: track 30.0 -> 48.7 mm
- net N-0000054 (its old number): track 11.6 -> 0.00 mm
- net N-0000066: track 11.2 -> 0.00 mm
- net N-0000067 (its old number): track 10.8 -> 0.00 mm
- net N-0000060 (its old number): track 6.58 -> 0.00 mm
- net N-0000067: track 44.8 -> 50.7 mm, vias 2 -> 0
- net N-0000061: track 0.00 -> 5.31 mm
- net N-0000069: track 0.00 -> 5.10 mm
- net N-0000062: track 10.1 -> 13.9 mm, vias 0 -> 1
- net N-0000059 (its old number): track 3.30 -> 0.00 mm
- net N-0000064: track 0.00 -> 2.66 mm
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Other:
- board text added: "Gain"
- board text added: "L R"
