File: PCB/Cabinas/Cabinas.sch (KiCad schematic (older format))
At the start: 110 parts, among them J1 JACK_ST_3SW, K1 CONN_3, M1 WTV020-SD, P1 CONN_2, P10 CONN_2, P11 CONN_2, P12 CONN_2, P13 DIN_5, P2 CONN_2, P3 CONN_2, P4 CONN_2, P5 CONN_2, P6 CONN_2, P7 CONN_2, P8 CONN_2, P9 CONN_2, Q1 MOSFET_N, Q10 MOSFET_N, Q11 MOSFET_N, Q12 MOSFET_N, Q2 MOSFET_N, Q3 MOSFET_N, Q4 MOSFET_N, Q5 MOSFET_N, Q6 MOSFET_N, Q7 MOSFET_N, Q8 MOSFET_N, Q9 MOSFET_N, SW1 PUSHBUTTON, SW10 PUSHBUTTON, SW11 PUSHBUTTON, SW12 PUSHBUTTON, SW2 PUSHBUTTON, SW3 PUSHBUTTON, SW4 PUSHBUTTON, SW5 PUSHBUTTON, SW6 PUSHBUTTON, SW7 PUSHBUTTON, SW8 PUSHBUTTON, SW9 PUSHBUTTON, U1 BTM, U2 7805, U3 TL072

Commit message: Rev 1.2
Rev 1.2
Parts:
- removed P1, P10, P11, P12, P2, P3, P4, P5, P6, P7, P8, P9: CONN_2, symbol CONN_2
- added C13: 470uF, ~, symbol CP1
- added GS1, GS2: GS3, symbol GS3
- added P1, P2, P3, P4, P5, P6, P7, P8: CONN_4, symbol CONN_4
- added U4, U5: 74HC595, ~, symbol 74HC595
Connections:
- net labels added: 1, 10, 11, 12, 2, 3, 4, 5, 6, 7, 8, 9, SR_CLK, SR_Input, SR_LCLK, SR_OE
- net labels removed: D10, D11, D12, D13, D2, D3, D4, D5, D6, D7, D8, D9, RST
- wire segments 375 -> 439
- no-connect marks 12 -> 30
Other:
- note added: "Grupo A/G"
- note added: "Grupo B/H"
- note added: "Grupo C/D"
- note added: "Grupo F/I"
- note added: "Shift register"
- moved on the sheet: A1, C1, C10, C11, C12, C2, C3, C4, C5, C6, C7, C8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

Commit message: BOM
BOM
Parts:
- removed U1: BTM, ~, symbol BTM
- added U1: BTM_2, ~, symbol BTM_2
Connections:
- wire segments 439 -> 437
Changed lines of the file:
@@
 encoding utf-8
 Sheet 1 1
-Title ""
+Title "Cabinas"
 Date "4 aug 2014"
 Rev "1.2"
-Comp ""
-Comment1 ""
+Comp "Hackerspace Cholula"
+Comment1 "04/08/2014"
 Comment2 ""
 Comment3 ""
@@
 MP3_CK
 $Comp
-L BTM U1
-U 1 1 538E36F5
-P 15400 5950
-F 0 "U1" V 16350 5600 60  0000 C CNN
-F 1 "BTM" V 16450 5750 60  0000 C CNN
-F 2 "~" H 15400 5950 60  0000 C CNN
-F 3 "~" H 15400 5950 60  0000 C CNN
-	1    15400 5950
-	0    -1   -1   0
-$EndComp
-$Comp
-L GND #PWR66
+L GND #PWR69
 U 1 1 538E3D93
-P 15150 4900
-F 0 "#PWR66" H 15150 4900 30  0001 C CNN
-F 1 "GND" H 15150 4830 30  0001 C CNN
-F 2 "" H 15150 4900 60  0000 C CNN
-F 3 "" H 15150 4900 60  0000 C CNN
-	1    15150 4900
+P 15200 5650
+F 0 "#PWR69" H 15200 5650 30  0001 C CNN
+F 1 "GND" H 15200 5580 30  0001 C CNN
+F 2 "" H 15200 5650 60  0000 C CNN
+F 3 "" H 15200 5650 60  0000 C CNN
+	1    15200 5650
 	1    0    0    -1
 $EndComp
-NoConn ~ 15300 5600
-Text GLabel 15100 5400 0    60   Output ~ 0
+Text GLabel 15000 5300 0    60   Output ~ 0
 A0 (RX)
 $Comp
@@
 	0    -1   -1   0
 $EndComp
-Text GLabel 13750 4600 0    60   Input ~ 0
+Text GLabel 15300 4500 2    60   Input ~ 0
 A1 (TX)
 $Comp
 L GND #PWR62
 U 1 1 538FE40B
-P 15300 4550
-F 0 "#PWR62" H 15300 4550 30  0001 C CNN
-F 1 "GND" H 15300 4480 30  0001 C CNN
-F 2 "" H 15300 4550 60  0000 C CNN
-F 3 "" H 15300 4550 60  0000 C CNN
-	1    15300 4550
+P 13700 4650
+F 0 "#PWR62" H 13700 4650 30  0001 C CNN
+F 1 "GND" H 13700 4580 30  0001 C CNN
+F 2 "" H 13700 4650 60  0000 C CNN
+F 3 "" H 13700 4650 60  0000 C CNN
+	1    13700 4650
 	1    0    0    -1
 $EndComp
-NoConn ~ 15300 5200
 $Comp
 L +5V #PWR67
 U 1 1 53908A8A
-P 14950 5250
-F 0 "#PWR67" H 14950 5340 20  0001 C CNN
-F 1 "+5V" H 14950 5340 30  0000 C CNN
-F 2 "" H 14950 5250 60  0000 C CNN
-F 3 "" H 14950 5250 60  0000 C CNN
-	1    14950 5250
+P 14500 5350
+F 0 "#PWR67" H 14500 5440 20  0001 C CNN
+F 1 "+5V" H 14500 5440 30  0000 C CNN
+F 2 "" H 14500 5350 60  0000 C CNN
+F 3 "" H 14500 5350 60  0000 C CNN
+	1    14500 5350
 	1    0    0    -1
 $EndComp
-Text Notes 13550 4750 0    60   ~ 0
+Text Notes 13350 4400 0    60   ~ 0
 Arduino - TX\nBTM - RX
-Text Notes 14500 5600 0    60   ~ 0
+Text Notes 14350 5700 0    60   ~ 0
 Arduino - RX\nBTM - TX
 $Comp
@@
 $EndComp
 $Comp
-L GND #PWR68
+L GND #PWR66
 U 1 1 53B35C66
 P 12250 5300
-F 0 "#PWR68" H 12250 5300 30  0001 C CNN
+F 0 "#PWR66" H 12250 5300 30  0001 C CNN
 F 1 "GND" H 12250 5230 30  0001 C CNN
 F 2 "" H 12250 5300 60  0000 C CNN
@@
 $EndComp
 $Comp
-L GND #PWR69
+L GND #PWR68
 U 1 1 53BD738B
 P 9500 5450
-F 0 "#PWR69" H 9500 5450 30  0001 C CNN
+F 0 "#PWR68" H 9500 5450 30  0001 C CNN
 F 1 "GND" H 9500 5380 30  0001 C CNN
 F 2 "" H 9500 5450 60  0000 C CNN
@@
 	13350 2500 13350 2300
 Wire Wire Line
-	15300 5100 15250 5100
-Wire Wire Line
-	15250 5100 15250 4850
-Wire Wire Line
-	15250 4850 15150 4850
-Wire Wire Line
-	15150 4850 15150 4900
-Wire Wire Line
-	15100 5400 15300 5400
-Wire Wire Line
 	14550 4500 14450 4500
 Wire Wire Line
-	14450 4500 14450 5500
-Wire Wire Line
 	14450 4600 14300 4600
 Wire Wire Line
@@
 Connection ~ 14450 4600
 Wire Wire Line
-	13800 4600 13750 4600
+	13700 4600 13800 4600
 Wire Wire Line
 	15050 4500 15300 4500
@@
 	15150 4700 15050 4700
 Connection ~ 14450 4700
-Wire Wire Line
-	15300 4500 15300 4550
 Connection ~ 15150 4500
 Wire Wire Line
-	15300 5300 14950 5300
-Wire Wire Line
-	14950 5300 14950 5250
-Wire Wire Line
-	14450 5500 15300 5500
-Wire Wire Line
 	11600 6450 11600 6400
 Wire Wire Line
@@
 Connection ~ 9800 2700
 Connection ~ 9650 3300
+Wire Wire Line
+	13700 4650 13700 4600
+$Comp
+L BTM_2 U1
+U 1 1 53DFD57F
+P 15500 5350
+F 0 "U1" H 15850 5000 60  0000 C CNN
+F 1 "BTM_2" H 15250 5100 60  0000 C CNN
+F 2 "~" H 14900 5450 60  0000 C CNN
+F 3 "~" H 14900 5450 60  0000 C CNN
+	1    15500 5350
+	0    -1   -1   0
+$EndComp
+Wire Wire Line
+	14450 4500 14450 5200
+Wire Wire Line
+	14450 5200 15300 5200
+Wire Wire Line
+	15300 5400 15200 5400
+Wire Wire Line
+	15200 5400 15200 5650
+Wire Wire Line
+	15000 5300 15300 5300
+Wire Wire Line
+	14500 5350 14500 5500
+Wire Wire Line
+	14500 5500 15300 5500
+NoConn ~ 15300 5600
+NoConn ~ 15300 5100
 $EndSCHEMATC

Commit message: PCB Rev 1.3
Parts:
- removed C11, C12: 1uF, ~, symbol CP1
- removed C8: 47uF, ~, symbol CP1
- removed ELEC1: ELECTRET_MIC_SUP, symbol ELECTRET_MIC_SUP
- removed GS1, GS2: GS3, symbol GS3
- removed J1: JACK_ST_3SW, ~, symbol JACK_ST_3SW
- removed JP1: JUMPER, symbol CONN_2
- removed R18, R19, R21, R22, R23, R24, R26: 10k, ~, symbol R
- removed R20: 270k, ~, symbol R
- removed R25: 2.2k, ~, symbol R
- removed U3: TL072, symbol TL072
- added D25: DIODE, ~, symbol DIODE
- added FB1: FILTER, ~, symbol FILTER
- added K2, TP1: CONN_3, symbol CONN_3
- added SW13, SW14, SW15: PUSHBUTTON, ~, symbol PUSHBUTTON
- added TP2, TP3: CONN_2, symbol CONN_2
Connections:
- net labels added: Next, Play, VCC
- net labels removed: Vbias
- wire segments 437 -> 419
- no-connect marks 30 -> 29
Other:
- note removed: "Mixing and amplifying"
- moved on the sheet: C1, C10, C2, C9, JP2, R15, R16, R17, REG1, U1, U2

Commit message: Rev 1.4
Parts:
- removed K1, K2: CONN_3, symbol CONN_3
- added C11: 0.022uF, ~, symbol C
- added C12, C16: 0.1uF, ~, symbol C
- added C14: 10uF, ~, symbol CP1
- added C15, C17: 270uF, ~, symbol CP1
- added C8: 0.22uF, ~, symbol C
- added J1, J2: JACK_ST, ~, symbol JACK_ST
- added P10, P9: CONN_2, symbol CONN_2
- added P11: CONN_6, symbol CONN_6
- added R18: 220, ~, symbol R
- added R19: 2.2k, ~, symbol R
- added R20: 10R, ~, symbol R
- added R21, R22, R23: R, ~, symbol R
- added R24, R25: 10k, ~, symbol R
- added RV1: 10k, ~, symbol POT
- added U3: LM386, ~, symbol LM386
- added U6: TL082, ~, symbol TL082
Connections:
- net labels added: +12P, MIC_PREAMP, Vbias
- wire segments 419 -> 481
Other:
- note added: "Digital PSU"
- note added: "LED PSU"
- note removed: "Alternate PSU"

Commit message: Rev 1.4
Other:
- note added: "Mic Preamp"
- note added: "Mixer/Preamp"
- note added: "Test Points"
- note added: "Virtual GND"
- moved on the sheet: C13, C3, C4, C5, C6, C7, J2, P11, R21, R22, R23, R24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

Commit message: Rev 1.5
Audio estereo
Parts:
- removed C10, C9: 1uF, ~, symbol CP1
- removed C3: 0.1uF, ~, symbol C
- removed M1: WTV020-SD, ~, symbol WTV020-SD
- removed P11: CONN_6, symbol CONN_6
- removed R23: R, ~, symbol R
- removed REG1: NPC1700, symbol NPC1700
- removed TP1: CONN_3, symbol CONN_3
- removed TP3: CONN_2, symbol CONN_2
- added A2: PROMINI, symbol PROMINI
- added K1, K2: CONN_3, symbol CONN_3
- added MP31: VS1053_ADAFRUIT, ~, symbol VS1053_ADAFRUIT
- added R26, R27, R28: 10k, ~, symbol R
- added R29, R30: R, ~, symbol R
- added RV2, RV3: 10k, ~, symbol POT
Connections:
- net labels added: LOUT, ROUT
- net labels removed: +3.3V, MP3_BUSY, MP3_CK, MP3_DATA, MP3_OUTPUT
- wire segments 481 -> 504
- no-connect marks 29 -> 23
Other:
- note added: "Audio"
- note added: "I2C"
- note added: "I2C and Button pad\nPower Supply"
- note added: "Mixer"
- note added: "Power"
- note removed: "3.3V Regulator"
- note removed: "I2C and Power Supply"
- note removed: "Mixer/Preamp"
- moved on the sheet: A1, C1, C11, C12, C13, C14, C15, C16, C17, C2, C4, C5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

Commit message: Firmware V3.0
Parts:
- removed C11: 0.022uF, ~, symbol C
- removed C15, C17: 270uF, ~, symbol CP1
- removed C16: 0.1uF, ~, symbol C
- removed C8: 0.22uF, ~, symbol C
- removed R20: 10R, ~, symbol R
- added C3, C8: 10uF, ~, symbol CP1
- added P11: CONN_2, symbol CONN_2
- C12: value 0.1uF -> 10pF
- R18: value 220 -> 0R
- R19: value 2.2k -> 100
Connections:
- wire segments 504 -> 505
Other:
- moved on the sheet: C12, C14, J1, K2, R19, RV1, U3

Commit message: REV 1.5
Codigo V3.0
Parts:
- R21, R22, R29, R30: value R -> 1k
Changed lines of the file:
@@
 Sheet 1 1
 Title "Cabinas"
-Date "26 jan 2015"
+Date "2 mar 2015"
 Rev "1.4"
 Comp "Hackerspace Cholula"
@@
 P 9150 9250
 F 0 "R22" V 9230 9250 40  0000 C CNN
-F 1 "R" V 9157 9251 40  0000 C CNN
+F 1 "1k" V 9157 9251 40  0000 C CNN
 F 2 "~" V 9080 9250 30  0000 C CNN
 F 3 "~" H 9150 9250 30  0000 C CNN
@@
 P 9150 8950
 F 0 "R21" V 9230 8950 40  0000 C CNN
-F 1 "R" V 9157 8951 40  0000 C CNN
+F 1 "1k" V 9157 8951 40  0000 C CNN
 F 2 "~" V 9080 8950 30  0000 C CNN
 F 3 "~" H 9150 8950 30  0000 C CNN
@@
 P 9150 10800
 F 0 "R30" V 9230 10800 40  0000 C CNN
-F 1 "R" V 9157 10801 40  0000 C CNN
+F 1 "1k" V 9157 10801 40  0000 C CNN
 F 2 "~" V 9080 10800 30  0000 C CNN
 F 3 "~" H 9150 10800 30  0000 C CNN
@@
 P 9150 10500
 F 0 "R29" V 9230 10500 40  0000 C CNN
-F 1 "R" V 9157 10501 40  0000 C CNN
+F 1 "1k" V 9157 10501 40  0000 C CNN
 F 2 "~" V 9080 10500 30  0000 C CNN
 F 3 "~" H 9150 10500 30  0000 C CNN
